File: TMC5160-LPHV.kicad_sch (KiCad schematic)
At the start: 15 parts, among them J1 StepStick Left, J2 StepStick Right, J3 StepStick Diag, Q1 DMT6018LDR, Q2 DMT6018LDR, Q3 DMT6018LDR, Q4 DMT6018LDR, U1 TMC5160A-TA

Commit message: switch to four-layer, minor improvements
Parts:
- Q1, Q2, Q3, Q4: Height 0.9 -> (none)
Changed lines of the file:
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@@
-			)
-		)
-		(property "Height" "0.9"
-			(at 120.65 464.77 0)
-			(effects
-				(font
-					(size 1.27 1.27)
-				)
-				(justify left top)
-				(hide yes)
 			)
 		)
@@
 			)
 		)
-		(property "Height" "0.9"
-			(at 120.65 500.33 0)
-			(effects
-				(font
-					(size 1.27 1.27)
-				)
-				(justify left top)
-				(hide yes)
-			)
-		)
 		(property "MPN" "DMT6018LDR-7"
 			(at 120.65 700.33 0)
@@
 			)
 		)
-		(property "Height" "0.9"
-			(at 120.65 482.55 0)
-			(effects
-				(font
-					(size 1.27 1.27)
-				)
-				(justify left top)
-				(hide yes)
-			)
-		)
 		(property "MPN" "DMT6018LDR-7"
 			(at 120.65 682.55 0)
@@
 				(hide yes)
 			)
-		)
-		(property "Height" "0.9"
-			(at 120.65 518.11 0)
-			(effects
-				(font
-					(size 1.27 1.27)
-				)
-				(justify left top)
-				(hide yes)
-			)
